File: pico.kicad_sch (KiCad schematic)
At the start: 46 parts, among them J16 USB_C_Receptacle_USB2.0_14P, J17 Conn_01x08, J19 Conn_01x10, J2 Conn_01x03_MountingPin, Q5 BSS138, Q6 BSS138, SW1 SW_MEC_5E, U15 RP2350B-QFN80, U18 W25Q128JVS, U24 MB85RS256B, Y3 12MHz

Commit message: Switched back to 2350A, rewired FPGA pins, maybe added some stuff? Idk.
Parts:
- removed BZ1: Buzzer, symbol Device:Buzzer
- removed C26, C27: 4.7uF, Capacitor_SMD:C_0402_1005Metric, symbol Device:C
- removed C29: 4.7u, Capacitor_SMD:C_0402_1005Metric, symbol Device:C
- removed C30, C31: 15p, Capacitor_SMD:C_0402_1005Metric, symbol Device:C
- removed C32: 100nF, Capacitor_SMD:C_0402_1005Metric, symbol Device:C
- removed D2: WS2812B, LED_SMD:LED_WS2812B_PLCC4_5.0x5.0mm_P3.2mm, symbol LED:WS2812B
- removed J16: USB_C_Receptacle_USB2.0_14P, Snapeda:1608_OSxx1608, symbol Connector:USB_C_Receptacle_USB2.0_14P
- removed J17: Conn_01x08, symbol Connector_Generic:Conn_01x08
- removed J19: Conn_01x10, symbol Connector_Generic:Conn_01x10
- removed J2: Conn_01x03_MountingPin, Connector_JST:JST_GH_SM03B-GHS-TB_1x03-1MP_P1.25mm_Horizontal, symbol Connector_Generic_MountingPin:Conn_01x03_MountingPin
- removed L3: L, symbol Device:L
- removed Q5, Q6: BSS138, Package_TO_SOT_SMD:SOT-23, symbol Transistor_FET:BSS138
- removed R13, R7: 27, Resistor_SMD:R_0402_1005Metric, symbol Device:R
- removed R22: 33, Resistor_SMD:R_0402_1005Metric, symbol Device:R
- removed R23, R25: 1k, Resistor_SMD:R_0402_1005Metric, symbol Device:R
- removed R24: 0, Resistor_SMD:R_0402_1005Metric, symbol Device:R
- removed R28, R29: 5.1K, Resistor_SMD:R_0402_1005Metric, symbol Device:R
- removed R30, R31: 100R, Resistor_SMD:R_0201_0603Metric, symbol Device:R
- removed R33, R35, R36: 10K, Resistor_SMD:R_0603_1608Metric_Pad0.98x0.95mm_HandSolder, symbol Device:R
- removed SW1: SW_MEC_5E, symbol Switch:SW_MEC_5E
- removed U15: RP2350B-QFN80, Package_DFN_QFN:QFN-80-1EP_10x10mm_P0.4mm_EP3.4x3.4mm, symbol RP2350x:RP2350B-QFN80
- removed U18: W25Q128JVS, Package_SO:SOIC-8_5.3x5.3mm_P1.27mm, symbol Memory_Flash:W25Q128JVS
- removed U24: MB85RS256B, Package_SO:SO-8_3.9x4.9mm_P1.27mm, symbol Memory_NVRAM:MB85RS256B
- removed Y3: 12MHz, Oscillator:Oscillator_SMD_Abracon_ASE-4Pin_3.2x2.5mm, symbol Device:Crystal_GND24
- added C39: 100nF, Capacitor_SMD:C_0402_1005Metric, symbol Device:C
- added C45, C46: 15p, Capacitor_SMD:C_0402_1005Metric, symbol Device:C
- added C47, C48: 4.7uF, Capacitor_SMD:C_0402_1005Metric, symbol Device:C
- added C49: 4.7u, Capacitor_SMD:C_0402_1005Metric, symbol Device:C
- added D13, D14, D8: LED, LED_SMD:LED_1206_3216Metric, symbol Device:LED
- added D4: WS2812B, LED_SMD:LED_WS2812B_PLCC4_5.0x5.0mm_P3.2mm, symbol LED:WS2812B
- added J11: Conn_01x03_MountingPin, Connector_JST:JST_GH_SM03B-GHS-TB_1x03-1MP_P1.25mm_Horizontal, symbol Connector_Generic_MountingPin:Conn_01x03_MountingPin
- added J14: USB_C_Receptacle_USB2.0_16P, Connector_USB:USB_C_Receptacle_GCT_USB4105-xx-A_16P_TopMnt_Horizontal, symbol Connector:USB_C_Receptacle_USB2.0_16P
- added J25: Conn_01x08, Connector_JST:JST_GH_BM08B-GHS-TBT_1x08-1MP_P1.25mm_Vertical, symbol Connector_Generic:Conn_01x08
- added L4: 3.3uH, Capacitor_SMD:C_0805_2012Metric_Pad1.18x1.45mm_HandSolder, symbol Device:L
- added Q8, Q9: BSS138, Package_TO_SOT_SMD:SOT-23, symbol Transistor_FET:BSS138
- added R10, R11, R4: 220, Resistor_SMD:R_0805_2012Metric_Pad1.20x1.40mm_HandSolder, symbol Device:R
- added R14, R15: 27, Resistor_SMD:R_0402_1005Metric, symbol Device:R
- added R27, R43: 1k, Resistor_SMD:R_0402_1005Metric, symbol Device:R
- added R42, R47, R50: 10K, Resistor_SMD:R_0603_1608Metric_Pad0.98x0.95mm_HandSolder, symbol Device:R
- added R44, R45: 100R, Resistor_SMD:R_0402_1005Metric_Pad0.72x0.64mm_HandSolder, symbol Device:R
- added R46: 33, Resistor_SMD:R_0402_1005Metric, symbol Device:R
- added R48, R49: 5.1K, Resistor_SMD:R_0402_1005Metric, symbol Device:R
- added SW5: SW_Push, Button_Switch_SMD:SW_Push_1P1T_NO_CK_KMR2, symbol Switch:SW_Push
- added U1: RP2350A-QFN60, Package_DFN_QFN:QFN-60-1EP_7x7mm_P0.4mm_EP3.4x3.4mm, symbol RP2350x:RP2350A-QFN60
- added U20: W25Q128JVS, Package_SO:SOIC-8_5.3x5.3mm_P1.27mm, symbol Memory_Flash:W25Q128JVS
- added U28: MB85RS256B, Package_SO:SO-8_3.9x4.9mm_P1.27mm, symbol Memory_NVRAM:MB85RS256B
- added Y4: 12MHz, Oscillator:Oscillator_SMD_Abracon_ASE-4Pin_3.2x2.5mm, symbol Device:Crystal_GND24
Connections:
- net +1V1: now also C48.1, L4.1, U1.23 (DVDD), U1.39 (DVDD), U1.50 (VREG_FB), U1.6 (DVDD)
- net +3V3: now also C39.2, C47.1, J25.7 (Pin_7), Q9.1 (G), R46.1, R47.1, U1.1 (IOVDD), U1.11 (IOVDD), U1.20 (IOVDD), U1.30 (IOVDD), U1.38 (IOVDD), U1.44 (ADC_AVDD), U1.45 (IOVDD), U1.49 (VREG_VIN), U1.53 (USB_OTP_VDD), U1.54 (QSPI_IOVDD), U20.8 (VCC), U28.3 (~{WP}), U28.7 (~{HOLD}), U28.8 (VDD)
- net +5V: now also D4.1 (VDD), R4.1, R50.2
- net ACTIVE: now also R10.1, U1.9 (GPIO6)
- net CAN_CS: now also U1.32 (GPIO20)
- net CAN_INT: now also U1.33 (GPIO21)
- net FPGA_CS: now also U1.8 (GPIO5)
- net GND: now also C39.1, C45.1, C46.1, C47.2, C48.2, C49.1, D13.1 (K), D14.1 (K), D4.3 (VSS), D8.1 (K), J11.2 (Pin_2), J11.MP (MountPin), J14.A1 (GND), J14.A12 (GND), J14.B1 (GND), J14.B12 (GND), J14.SH (SHIELD), J25.8 (Pin_8), Q8.2 (S), R42.1, R48.2, R49.1, SW5.1, U1.47 (VREG_PGND), U1.61 (GND), U20.4 (GND), U28.4 (GND), Y4.2 (G), Y4.4 (G)
- net IMU_INT: now also U1.29 (GPIO18)
- net MASTER_INT: now also U1.17 (GPIO13)
- net MISO_INT: now also U1.7 (GPIO4), U28.2 (SO)
- net MISO_OUT: now also U1.16 (GPIO12)
- net MOSI_INT: now also U1.5 (GPIO3), U28.5 (SI)
- net MOSI_OUT: now also U1.15 (GPIO11)
- net RPI_READY: now also U1.10 (GPIO7)
- net RUN: now also Q8.1 (G), R42.2
- net SCK_INT: now also U1.4 (GPIO2), U28.6 (SCK)
- net SCK_OUT: now also U1.14 (GPIO10)
- net SCL: now also R11.1, U1.3 (GPIO1)
- net SCL_OUT: now also U1.19 (GPIO15)
- net SDA: now also U1.2 (GPIO0)
- net SDA_OUT: now also U1.18 (GPIO14)
- net UART_RX: now also U1.13 (GPIO9)
- net UART_TX: now also U1.12 (GPIO8)
- net VUSB: now also J14.A4 (VBUS), J14.A9 (VBUS), J14.B4 (VBUS), J14.B9 (VBUS)
- new net: D14.2 (A), R11.2
- new net: J14.B5 (CC2), R48.1
- new net: J14.A5 (CC1), R49.2
- new net: J14.A6 (D+), J14.B6 (D+), R14.2
- new net: J14.A7 (D-), J14.B7 (D-), R15.1
- new net: Q9.2 (S), U1.35 (GPIO23)
- new net: D4.4 (DIN), Q9.3 (D), R50.1
- new net: D13.2 (A), R4.2
- new net: C46.2, R43.1, Y4.3
- new net: R43.2, U1.22 (XOUT)
- new net: R45.1, U1.25 (SWDIO)
- new net: J11.3 (Pin_3), R45.2
- new net: J25.1 (Pin_1), U1.36 (GPIO24)
- new net: J25.2 (Pin_2), U1.37 (GPIO25)
- new net: J25.3 (Pin_3), U1.40 (GPIO26_ADC0)
- new net: J25.4 (Pin_4), U1.41 (GPIO27_ADC1)
- new net: J25.5 (Pin_5), U1.42 (GPIO28_ADC2)
- new net: J25.6 (Pin_6), U1.43 (GPIO29_ADC3)
- new net: C45.2, U1.21 (XIN), Y4.1
- new net: R44.2, U1.24 (SWCLK)
- new net: Q8.3 (D), R47.2, U1.26 (RUN)
- new net: U1.34 (GPIO22), U28.1 (~{CS})
- new net: C49.2, R46.2, U1.46 (VREG_AVDD)
- new net: L4.2, U1.48 (VREG_LX)
- new net: R15.2, U1.51 (USB_DM)
- new net: R14.1, U1.52 (USB_DP)
- new net: U1.55 (QSPI_SD3), U20.7 (~{HOLD}/~{RESET}/IO_{3})
- new net: U1.56 (QSPI_SCLK), U20.6 (CLK)
- new net: U1.57 (QSPI_SD0), U20.5 (DI/IO_{0})
- new net: U1.58 (QSPI_SD2), U20.3 (~{WP}/IO_{2})
- new net: U1.59 (QSPI_SD1), U20.2 (DO/IO_{1})
- new net: R27.2, U1.60 (QSPI_SS), U20.1 (~{CS})
- new net: R27.1, SW5.2
- new net: J11.1 (Pin_1), R44.1
- new net: D8.2 (A), R10.2
- new net PPS: U1.31 (GPIO19)
- new net RX_INT: U1.28 (GPIO17)
- new net TX_INT: U1.27 (GPIO16)
- no-connect marks 1 -> 3
Other:
- note added: "TODO: figure out what to do with all these leftover pins! What a problem to have..."
- note added: "UART0"
- note added: "UART1"
