File: psu.kicad_sch (KiCad schematic)
At the start: 14 parts, among them J1 Screw_Terminal_01x02, J11 Screw_Terminal_01x02, U12 XL1509-3.3, U13 XL1509-5.0, U14 INA219AxD

Commit message: Implementing just so much stuff. RP2350B on board, new sensors, PSU magic, buncha stuff
Parts:
- removed C7, C8: 180uF, Capacitor_SMD:CP_Elec_10x10, symbol Device:C_Polarized_US
- removed D4, D5: 1N5820, Diode_THT:D_DO-201AD_P15.24mm_Horizontal, symbol Diode:1N5820
- removed U12: XL1509-3.3, Package_SO:SOIC-8_3.9x4.9mm_P1.27mm, symbol Regulator_Switching:XL1509-3.3
- removed U13: XL1509-5.0, Package_SO:SOIC-8_3.9x4.9mm_P1.27mm, symbol Regulator_Switching:XL1509-5.0
- added C33: 47uF, Capacitor_SMD:C_Elec_4x5.4, symbol Device:C
- added C34, C35, C36, C8: 22uF, Capacitor_SMD:C_0603_1608Metric, symbol Device:C
- added C37: 100nF, Capacitor_SMD:C_0402_1005Metric, symbol Device:C
- added C38, C7: 100nF, Capacitor_SMD:C_0603_1608Metric, symbol Device:C
- added D5: SMAJ18A, Diode_SMD:D_SMA, symbol Diode:SMAJ18A
- added Q1: DMP3099L, Package_TO_SOT_SMD:SOT-23, symbol Transistor_FET:DMP3099L
- added R26: 33K, Resistor_SMD:R_0402_1005Metric, symbol Device:R
- added R27: 10K, Resistor_SMD:R_0402_1005Metric, symbol Device:R
- added R32: 100K, Resistor_SMD:R_0402_1005Metric, symbol Device:R
- added U20: AP63203WU, Package_TO_SOT_SMD:TSOT-23-6, symbol Regulator_Switching:AP63203WU
- added U21: AP63205WU, Package_TO_SOT_SMD:TSOT-23-6, symbol Regulator_Switching:AP63205WU
- added U22: TPS2116DRL, Package_TO_SOT_SMD:SOT-583-8, symbol Power_Management:TPS2116DRL
- C1: value 105uF -> 10uF; footprint Capacitor_SMD:C_0603_1608Metric -> Capacitor_SMD:C_0805_2012Metric
- C6: footprint Capacitor_SMD:CP_Elec_10x10 -> Capacitor_SMD:CP_Elec_6.3x5.4_Nichicon
- L1, L2: value 68uH -> 4.7uH; footprint (none) -> Inductor_SMD:L_0805_2012Metric
- R14: footprint Resistor_SMD:R_2512_6332Metric -> Resistor_SMD:R_2816_7142Metric_Pad3.20x4.45mm_HandSolder
Connections:
- net +3V3: now also L2.2, C35.1, C36.1, U20.1 (FB); no longer L1.2
- net +5V: now also U20.2 (EN), U20.3 (IN), U22.2 (VOUT), U22.7 (VOUT); no longer L2.2
- net at C1.1, C6.1, R14.2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: now also U21.2 (EN), U21.3 (IN); no longer J11.2 (Pin_2)
- net at L1.1: now also C7.2, U21.5 (SW)
- net at L2.1: now also C38.2, U20.5 (SW)
- net +BATT: no longer names the net of R14.1, U14.8 (IN+)
- net +BATT: now also D5.1 (A1), Q1.2 (S); no longer J1.2 (Pin_2)
- net -BATT renamed GND
- net GND: now also C34.2, C35.2, C36.2, C8.2, R27.1, R32.2, U20.4 (GND), U21.4 (GND), U22.1 (GND)
- new net: C34.1, C8.1, L1.2, U21.1 (FB), U22.6 (VIN2)
- new net: J1.2 (Pin_2), J11.2 (Pin_2), Q1.3 (D)
- new net: D5.2 (A2), Q1.1 (G), R32.1
- new net: C38.1, U20.6 (BST)
- new net: R26.2, R27.2, U22.4 (PR1)
- new net: C7.1, U21.6 (BST)
- new net MODE_V: U22.8 (ST)
- new net VUSB: R26.1, U22.3 (VIN1), U22.5 (MODE)

Commit message: Switched back to 2350A, rewired FPGA pins, maybe added some stuff? Idk.
Parts:
- added C39: 100nF, Capacitor_SMD:C_0603_1608Metric, symbol Device:C
- added L4: 4.7uH, Inductor_SMD:L_0805_2012Metric, symbol Device:L
Connections:
- net +3V3: now also L4.1; no longer L2.2
- net GND: no longer C35.2, C36.2, U20.4 (GND)
- net at C38.2, L2.1: no longer U20.5 (SW)
- net at U20.6 (BST): now also C39.1; no longer C38.1
- new net: C39.2, L4.2, U20.5 (SW)
- new net: C35.2, C36.2, U20.4 (GND)
Other:
- moved on the sheet: C33, C34, C35, C36, C37, C38, C7, C8, D5, J1, J11, L1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
