File: titanRIO.kicad_pcb (KiCad board)
At the start: 4 copper layers, 85 parts, among them J1 Screw_Terminal_01x02, J10 Conn_01x04, J11 Screw_Terminal_01x02, J12 Conn_01x10, J13 Conn_01x10, J14 Conn_01x10, J15 Screw_Terminal_01x02, J18 Screw_Terminal_01x02, J20 Conn_01x10, J3 Conn_01x05, J4 Conn_02x02_Odd_Even, J5 Screw_Terminal_01x02, J6 Conn_01x04, J7 Screw_Terminal_01x02, J8 Conn_01x12, J9 Conn_01x05, Q2 BSS138, Q3 BSS138, Q4 BSS138, SW2 SW_DIP_x03, SW3 SW_Push, U1 Tang_Nano_20K, U11 74LVC2G08, U12 XL1509-3.3, U13 XL1509-5.0, U14 INA219AxD, U15 RP2350B-QFN80, U16 74LVC1G175, U17 74HC123, U2 TCAN332G, U3 MCP2518FD-xQBB, U4 PCA9685BS, U5 SN74LVC8T245PWR, U6 SN74LVC8T245PWR, Y1 Crystal, Y2 SG-3031CM

Commit message: Switched back to 2350A, rewired FPGA pins, maybe added some stuff? Idk.
Parts:
- removed A1: RaspberryPi_Pico, Module:RaspberryPi_Pico_Common_Unspecified
- removed C1: 105uF, Capacitor_SMD:C_0201_0603Metric_Pad0.64x0.40mm_HandSolder
- removed C6: 470uF, Capacitor_SMD:CP_Elec_6.3x5.4_Nichicon
- removed C7, C8: 180uF, Capacitor_SMD:CP_Elec_6.3x5.4_Nichicon
- removed D1: WS2812B, LED_SMD:LED_WS2812B_PLCC4_5.0x5.0mm_P3.2mm
- removed D2: QLS6B-FKW, LED_SMD:LED_Cree-PLCC6_4.7x1.5mm
- removed D8: SS32, Diode_SMD:D_SMA
- removed J1, J11: Screw_Terminal_01x02, TerminalBlock_Phoenix:TerminalBlock_Phoenix_MPT-0,5-2-2.54_1x02_P2.54mm_Horizontal
- removed J14: Conn_01x10, Connector_JST:JST_GH_BM10B-GHS-TBT_1x10-1MP_P1.25mm_Vertical
- removed J8: Conn_01x12, Connector_JST:JST_GH_BM12B-GHS-TBT_1x12-1MP_P1.25mm_Vertical
- removed JP2: SolderJumper_2_Open, Jumper:SolderJumper-2_P1.3mm_Open_TrianglePad1.0x1.5mm
- removed L1: 68uH, Inductor_SMD:L_Bourns-SRU8028_8.0x8.0mm
- removed Q3: BSS138, Package_TO_SOT_SMD:SOT-23
- removed R1, R2, R3: 220, Resistor_SMD:R_0805_2012Metric_Pad1.20x1.40mm_HandSolder
- removed R10, R11, R15, R4: 10K, Resistor_SMD:R_0603_1608Metric_Pad0.98x0.95mm_HandSolder
- removed R14: 0.1, Resistor_SMD:R_2816_7142Metric_Pad3.20x4.45mm_HandSolder
- removed U1: Tang_Nano_20K, 0my_project:DIP-40_TangNano20K
- removed U13: XL1509-5.0, Package_SO:SOIC-8_3.9x4.9mm_P1.27mm
- added BZ2: Buzzer, Buzzer_Beeper:Buzzer_12x9.5RM7.6, F.Cu at (157.5, 29.9)
- added C26: 100nF, Capacitor_SMD:C_0402_1005Metric, F.Cu at (260.6, 26.6)
- added C27: 100nF, Capacitor_SMD:C_0402_1005Metric, F.Cu at (260.6, 28.5)
- added C29: 10u, Capacitor_SMD:C_0402_1005Metric, F.Cu at (253.0, 26.9)
- added C30: 100nF, Capacitor_SMD:C_0402_1005Metric, F.Cu at (260.6, 32.5)
- added C31: 100nF, Capacitor_SMD:C_0402_1005Metric, F.Cu at (260.6, 34.4)
- added C32: 100nF, Capacitor_SMD:C_0402_1005Metric, F.Cu at (263.5, 26.6)
- added C33: 470uF, Capacitor_SMD:CP_Elec_6.3x5.4_Nichicon, F.Cu at (260.9, 107.2)
- added C34: 10u, Capacitor_SMD:C_0402_1005Metric, F.Cu at (80.5, 145.5)
- added C35: 10u, Capacitor_SMD:C_0402_1005Metric, F.Cu at (80.5, 142.0)
- added C36: 10u, Capacitor_SMD:C_0402_1005Metric, F.Cu at (93.0, 136.0)
- added C37: 10uF, Capacitor_SMD:C_0805_2012Metric, F.Cu at (259.9, 98.8)
- added C38: 22uF, Capacitor_SMD:C_0603_1608Metric, F.Cu at (239.3, 117.3)
- added C40: 100nF, Capacitor_SMD:C_0603_1608Metric, F.Cu at (238.8, 113.3)
- added C41: 22uF, Capacitor_SMD:C_0603_1608Metric, F.Cu at (235.3, 117.3)
- added C42: 100nF, Capacitor_SMD:C_0603_1608Metric, F.Cu at (239.8, 106.3)
- added C43: 22uF, Capacitor_SMD:C_0603_1608Metric, F.Cu at (236.3, 109.8)
- added C44: 22uF, Capacitor_SMD:C_0603_1608Metric, F.Cu at (239.8, 109.8)
- added C50: 100nF, Capacitor_SMD:C_0402_1005Metric, F.Cu at (238.0, 62.0)
- added C51: 4.7uF, Capacitor_SMD:C_0402_1005Metric, F.Cu at (230.2, 53.4)
- added C52: 15p, Capacitor_SMD:C_0402_1005Metric, F.Cu at (230.4, 35.5)
- added C53: 15p, Capacitor_SMD:C_0402_1005Metric, F.Cu at (230.4, 41.0)
- added C54: 4.7uF, Capacitor_SMD:C_0402_1005Metric, F.Cu at (230.2, 51.9)
- added C55: 4.7u, Capacitor_SMD:C_0402_1005Metric, F.Cu at (238.0, 50.5)
- added C56: 100nF, Capacitor_SMD:C_0402_1005Metric, F.Cu at (263.5, 28.5)
- added C57: 100nF, Capacitor_SMD:C_0402_1005Metric, F.Cu at (263.5, 30.5)
- added C58: 100nF, Capacitor_SMD:C_0402_1005Metric, F.Cu at (263.5, 32.5)
- added C59: 100nF, Capacitor_SMD:C_0402_1005Metric, F.Cu at (263.5, 34.4)
- added C60: 100nF, Capacitor_SMD:C_0402_1005Metric, F.Cu at (253.0, 30.5)
- added C61: 100nF, Capacitor_SMD:C_0402_1005Metric, F.Cu at (253.0, 32.5)
- added C62: 100nF, Capacitor_SMD:C_0402_1005Metric, F.Cu at (253.0, 34.4)
- added D15: LED, LED_SMD:LED_1206_3216Metric, F.Cu at (62.0, 19.1)
- added D16: LED, LED_SMD:LED_1206_3216Metric, F.Cu at (62.0, 25.1)
- added D17: SS32, Diode_SMD:D_SMA, F.Cu at (207.0, 17.5)
- added D5: WS2812B, LED_SMD:LED_WS2812B_PLCC4_5.0x5.0mm_P3.2mm, F.Cu at (219.5, 17.0)
- added F1: 2920L600/24SL, Fuse:Fuse_2920_7451Metric, F.Cu at (238.4, 98.3)
- added J16: Conn_01x03_MountingPin, Connector_JST:JST_GH_SM03B-GHS-TB_1x03-1MP_P1.25mm_Horizontal, F.Cu at (234.0, 18.5)
- added J17: USB_C_Receptacle_USB2.0_16P, Connector_USB:USB_C_Receptacle_GCT_USB4105-xx-A_16P_TopMnt_Horizontal, F.Cu at (249.4, 18.4)
- added J21: Conn_01x08, Connector_JST:JST_GH_BM08B-GHS-TBT_1x08-1MP_P1.25mm_Vertical, F.Cu at (27.2, 18.6)
- added J22: Conn_01x02, Connector_JST:JST_PH_B2B-PH-K_1x02_P2.00mm_Vertical, F.Cu at (31.9, 30.1)
- added J23: Screw_Terminal_01x02, TerminalBlock_Phoenix:TerminalBlock_Phoenix_MPT-0,5-2-2.54_1x02_P2.54mm_Horizontal, F.Cu at (261.0, 117.5)
- added J24: Conn_01x12, Connector_JST:JST_GH_BM12B-GHS-TBT_1x12-1MP_P1.25mm_Vertical, F.Cu at (94.0, 18.0)
- added J26: Conn_01x08, Connector_JST:JST_GH_BM08B-GHS-TBT_1x08-1MP_P1.25mm_Vertical, F.Cu at (280.5, 45.0)
- added JP4: SolderJumper_2_Open, Jumper:SolderJumper-2_P1.3mm_Open_TrianglePad1.0x1.5mm, F.Cu at (32.7, 24.6)
- added JP6: SolderJumper_2_Open, Jumper:SolderJumper-2_P1.3mm_Open_TrianglePad1.0x1.5mm, F.Cu at (98.5, 24.5)
- added L5: 4.7uH, Inductor_SMD:L_0805_2012Metric, F.Cu at (248.8, 110.4)
- added L6: 3.3uH, Capacitor_SMD:C_0805_2012Metric_Pad1.18x1.45mm_HandSolder, F.Cu at (233.5, 52.0)
- added Q10: BSS138, Package_TO_SOT_SMD:SOT-23, F.Cu at (227.9, 30.1)
- added Q11: BSS138, Package_TO_SOT_SMD:SOT-23, F.Cu at (221.0, 22.9)
- added Q7: BSS138, Package_TO_SOT_SMD:SOT-23, F.Cu at (87.0, 157.0)
- added R13: 220, Resistor_SMD:R_0805_2012Metric_Pad1.20x1.40mm_HandSolder, F.Cu at (57.0, 22.1)
- added R22: 220, Resistor_SMD:R_0805_2012Metric_Pad1.20x1.40mm_HandSolder, F.Cu at (57.0, 25.0)
- added R23: 27, Resistor_SMD:R_0402_1005Metric, F.Cu at (248.5, 24.5)
- added R24: 27, Resistor_SMD:R_0402_1005Metric, F.Cu at (250.0, 24.5)
- added R26: 10K, Resistor_SMD:R_0603_1608Metric_Pad0.98x0.95mm_HandSolder, F.Cu at (177.8, 116.1)
- added R28: 1k, Resistor_SMD:R_0402_1005Metric, F.Cu at (244.5, 63.0)
- added R34: 100K, Resistor_SMD:R_0402_1005Metric, F.Cu at (248.9, 100.3)
- added R37: 0.1, Resistor_SMD:R_2816_7142Metric_Pad3.20x4.45mm_HandSolder, F.Cu at (253.9, 97.8)
- added R38: 33K, Resistor_SMD:R_0402_1005Metric, F.Cu at (251.8, 115.3)
- added R39: 10K, Resistor_SMD:R_0402_1005Metric, F.Cu at (251.8, 113.3)
- added R40: 10K, Resistor_SMD:R_0603_1608Metric_Pad0.98x0.95mm_HandSolder, F.Cu at (87.0, 154.0)
- added R41: 10K, Resistor_SMD:R_0603_1608Metric_Pad0.98x0.95mm_HandSolder, F.Cu at (84.0, 157.5)
- added R51: 10K, Resistor_SMD:R_0603_1608Metric_Pad0.98x0.95mm_HandSolder, F.Cu at (223.9, 30.1)
- added R52: 10K, Resistor_SMD:R_0603_1608Metric_Pad0.98x0.95mm_HandSolder, F.Cu at (231.4, 29.1)
- added R53: 100R, Resistor_SMD:R_0402_1005Metric_Pad0.72x0.64mm_HandSolder, F.Cu at (235.2, 23.5)
- added R54: 100R, Resistor_SMD:R_0402_1005Metric_Pad0.72x0.64mm_HandSolder, F.Cu at (233.2, 23.5)
- added R55: 1k, Resistor_SMD:R_0402_1005Metric, F.Cu at (226.9, 39.0)
- added R56: 33, Resistor_SMD:R_0402_1005Metric, F.Cu at (236.0, 49.0)
- added R57: 5.1K, Resistor_SMD:R_0402_1005Metric, F.Cu at (247.0, 24.0)
- added R58: 5.1K, Resistor_SMD:R_0402_1005Metric, F.Cu at (251.5, 24.0)
- added R59: 10K, Resistor_SMD:R_0603_1608Metric_Pad0.98x0.95mm_HandSolder, F.Cu at (225.0, 18.5)
- added R7: 220, Resistor_SMD:R_0805_2012Metric_Pad1.20x1.40mm_HandSolder, F.Cu at (57.0, 19.1)
- added SW6: SW_Push, Button_Switch_SMD:SW_Push_1P1T_NO_CK_KMR2, F.Cu at (241.6, 65.8)
- added U19: DAC6578xPW, Package_SO:TSSOP-16_4.4x5mm_P0.65mm, F.Cu at (21.5, 27.2)
- added U21: W25Q128JVS, Package_SO:SOIC-8_5.3x5.3mm_P1.27mm, F.Cu at (241.5, 58.5)
- added U23: INA219AxD, Package_SO:SOIC-8_3.9x4.9mm_P1.27mm, F.Cu at (246.3, 121.9)
- added U25: AP63203WU, Package_TO_SOT_SMD:TSOT-23-6, F.Cu at (243.9, 108.7)
- added U26: AP63205WU, Package_TO_SOT_SMD:TSOT-23-6, F.Cu at (243.9, 113.3)
- added U27: TPS2116DRL, Package_TO_SOT_SMD:SOT-583-8, F.Cu at (249.0, 114.0)
- added U29: MB85RS256B, Package_SO:SO-8_3.9x4.9mm_P1.27mm, F.Cu at (222.4, 46.1)
- added Y5: 12MHz, Oscillator:Oscillator_SMD_Abracon_ASE-4Pin_3.2x2.5mm, F.Cu at (230.4, 38.2)
- C10: footprint Capacitor_SMD:C_0201_0603Metric_Pad0.64x0.40mm_HandSolder -> Capacitor_SMD:C_0603_1608Metric
- C11: footprint Capacitor_SMD:C_0201_0603Metric_Pad0.64x0.40mm_HandSolder -> Capacitor_SMD:C_0603_1608Metric_Pad1.08x0.95mm_HandSolder
- C12, C13, C14, C2, C3, C4, C5: footprint Capacitor_SMD:C_0201_0603Metric_Pad0.64x0.40mm_HandSolder -> Capacitor_SMD:C_0402_1005Metric_Pad0.74x0.62mm_HandSolder
- D7: value SS32 -> SMAJ18A
- D9: value SS32 -> LED; footprint Diode_SMD:D_SMA -> LED_SMD:LED_1206_3216Metric
- J3: value Conn_01x05 -> Screw_Terminal_01x02; footprint Connector_JST:JST_GH_BM05B-GHS-TBT_1x05-1MP_P1.25mm_Vertical -> TerminalBlock_Phoenix:TerminalBlock_Phoenix_MPT-0,5-2-2.54_1x02_P2.54mm_Horizontal
- L2: value 68uH -> 4.7uH; footprint Inductor_SMD:L_Bourns-SRU8028_8.0x8.0mm -> Inductor_SMD:L_0805_2012Metric
- Q2: value BSS138 -> DMP3099L
- R5: footprint Resistor_SMD:R_1812_4532Metric_Pad1.30x3.40mm_HandSolder -> Resistor_SMD:R_1812_4532Metric
- U12: value XL1509-3.3 -> SAM-M8Q; footprint Package_SO:SOIC-8_3.9x4.9mm_P1.27mm -> RF_GPS:ublox_SAM-M8Q
- U14: value INA219AxD -> RP2350A-QFN60; footprint Package_SO:SOIC-8_3.9x4.9mm_P1.27mm -> Package_DFN_QFN:QFN-60-1EP_7x7mm_P0.4mm_EP3.4x3.4mm
- U15: value RP2350B-QFN80 -> Tang_Nano_20K; footprint Package_DFN_QFN:QFN-80-1EP_10x10mm_P0.4mm_EP3.4x3.4mm -> 0my_project:DIP-40_TangNano20K
- Y1: value Crystal -> 20mHz; footprint Crystal:Crystal_SMD_5032-2Pin_5.0x3.2mm -> Inductor_SMD:L_1008_2520Metric_Pad1.43x2.20mm_HandSolder
- moved U14 226.7 mm to (241.1, 45.5), turned to 180 degrees
- moved U8 223.8 mm to (23.5, 98.2), turned to 0 degrees
- moved J18 221.4 mm to (23.2, 142.5), turned to 0 degrees
- moved U7 219.6 mm to (23.5, 109.8), turned to 0 degrees
- moved U10 218.4 mm to (23.5, 132.8), turned to 0 degrees
- moved U9 217.7 mm to (23.5, 121.3), turned to 0 degrees
- moved D7 198.7 mm to (249.4, 103.8), turned to 180 degrees
- moved U4 188.7 mm to (38.2, 118.1), turned to -90 degrees
- moved L2 187.3 mm to (248.8, 107.7), turned to 0 degrees
- moved J9 161.7 mm to (41.4, 193.7)
- moved J10 161.7 mm to (30.1, 193.7)
- moved J6 161.7 mm to (19.1, 193.7)
- moved R8 161.7 mm to (18.8, 186.1)
- moved R9 161.7 mm to (18.8, 188.1)
- moved BNO08x1 154.0 mm to (43.5, 79.8)
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Connections:
- D7 pad 1: Net-(D7-K) -> Net-(D7-A1)
- D7 pad 2: GND -> Net-(D7-A2)
- D9 pad 1: Net-(D9-K) -> GND
- D9 pad 2: +5V -> Net-(D9-A)
- J3 pad 1: Net-(A1-ADC_VREF) -> GND
- JP3 pad 1: Net-(JP3-A) -> +3V3
- JP3 pad 2: WDI_MASTER -> Net-(JP3-B)
- L2 pad 2: +5V -> /5V_REG
- Q2 pad 1: +3V3 -> Net-(D7-A2)
- Q2 pad 2: Net-(Q2-S) -> Net-(D7-A1)
- SW2 pad 6: Net-(R15-Pad2) -> Net-(U17B-Q)
- U11 pad 6: Net-(R15-Pad2) -> Net-(U17B-Q)
- U12 pad 1: Net-(U12-VIN) -> GND
- U12 pad 2: Net-(D7-K) -> +3V3
- U12 pad 7: GND -> PPS
- U12 pad 8: GND -> unconnected-(U12-~{SAFEBOOT}-Pad8)
- U14 pad 2: +3V3 -> SDA
- U14 pad 3: SDA_OUT -> SCL
- U14 pad 4: SCL_OUT -> SCK_INT
- U14 pad 5: +3V3 -> MOSI_INT
- U14 pad 6: GND -> +1V1
- U14 pad 7: Net-(U12-VIN) -> MISO_INT
- U14 pad 8: Net-(J1-Pin_2) -> FPGA_CS
- U15 pad 1: unconnected-(U15-GPIO4-Pad1) -> ENC3A
- U15 pad 10: unconnected-(U15-DVDD-Pad10) -> B1_3
- U15 pad 11: unconnected-(U15-GPIO12-Pad11) -> B1_4
- U15 pad 12: unconnected-(U15-GPIO13-Pad12) -> B1_5
- U15 pad 13: unconnected-(U15-GPIO14-Pad13) -> B1_6
- U15 pad 14: unconnected-(U15-GPIO15-Pad14) -> B1_7
- U15 pad 15: unconnected-(U15-IOVDD-Pad15) -> FPGA_SIG0
- U15 pad 16: unconnected-(U15-GPIO16-Pad16) -> FPGA_SIG1
- U15 pad 17: unconnected-(U15-GPIO17-Pad17) -> ~{ACTIVE}
- U15 pad 18: unconnected-(U15-GPIO18-Pad18) -> ~{PPS}
- U15 pad 2: unconnected-(U15-GPIO5-Pad2) -> ENC4B
- U15 pad 20: unconnected-(U15-GPIO20-Pad20) -> GND
- U15 pad 21: unconnected-(U15-GPIO21-Pad21) -> ENC2B
- U15 pad 22: unconnected-(U15-GPIO22-Pad22) -> ENC2A
- U15 pad 23: unconnected-(U15-GPIO23-Pad23) -> ENC1B
- U15 pad 24: unconnected-(U15-IOVDD-Pad24) -> ENC1A
- U15 pad 26: unconnected-(U15-GPIO25-Pad26) -> GND
- U15 pad 28: unconnected-(U15-GPIO27-Pad28) -> B0_3
- U15 pad 29: unconnected-(U15-IOVDD-Pad29) -> B0_2
- U15 pad 3: unconnected-(U15-GPIO6-Pad3) -> ENC4A
- U15 pad 30: unconnected-(U15-XIN-Pad30) -> B0_7
- U15 pad 31: unconnected-(U15-XOUT-Pad31) -> B0_6
- U15 pad 32: unconnected-(U15-DVDD-Pad32) -> B0_5
- U15 pad 33: unconnected-(U15-SWCLK-Pad33) -> B0_4
- U15 pad 34: unconnected-(U15-SWDIO-Pad34) -> B0_0
- U15 pad 35: unconnected-(U15-RUN-Pad35) -> B0_1
- U15 pad 36: unconnected-(U15-GPIO28-Pad36) -> SCK_INT
- U15 pad 37: unconnected-(U15-GPIO29-Pad37) -> MISO_INT
- U15 pad 38: unconnected-(U15-GPIO30-Pad38) -> MOSI_INT
- U15 pad 39: unconnected-(U15-GPIO31-Pad39) -> GND
- U15 pad 4: unconnected-(U15-GPIO7-Pad4) -> ENC3B
- U15 pad 40: unconnected-(U15-GPIO32-Pad40) -> Net-(D17-K)
- U15 pad 5: unconnected-(U15-IOVDD-Pad5) -> B1_0
- U15 pad 6: unconnected-(U15-GPIO8-Pad6) -> Net-(BZ2-+)
- U15 pad 7: unconnected-(U15-GPIO9-Pad7) -> FPGA_CS
- U15 pad 8: unconnected-(U15-GPIO10-Pad8) -> B1_1
- U15 pad 9: unconnected-(U15-GPIO11-Pad9) -> B1_2
- U17 pad 10: Net-(JP3-A) -> WDI_MASTER
Routing:
- net +3V3: track 230.1 -> 177.4 mm
- net (no net): track 0.00 -> 50.3 mm
- net Net-(R15-Pad2): track 50.3 -> 0.00 mm, vias 2 -> 0
- net Net-(U12-VIN): track 50.2 -> 0.00 mm
- net GND: track 356.8 -> 310.1 mm
- net +5V: track 35.3 -> 0.00 mm
- net Net-(J1-Pin_2): track 28.9 -> 0.00 mm
- net Net-(D7-K): track 14.3 -> 0.00 mm
- net Net-(A1-GPIO27_ADC1): track 12.7 -> 0.00 mm
- net Net-(J23-Pin_2): track 12.2 -> 0.00 mm
- net VUSB: track 0.00 -> 6.79 mm
- net Net-(U26-SW): track 4.91 -> 0.00 mm
- net Net-(A1-AGND): track 4.64 -> 0.00 mm
- net Net-(J17-D--PadA7): track 0.00 -> 4.63 mm
- net PPS: track 0.00 -> 4.52 mm
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Other:
- copper layers 4 -> 2
- board text added: "PSU"
- board text added: "Pico"
- board text removed: "ADC"
- board text removed: "Harness"
- board text removed: "IO"

Commit message: PCB Design initialized. And mostly done tbf
Parts:
- removed C33: 470uF, Capacitor_SMD:CP_Elec_6.3x5.4_Nichicon
- removed C35, C36: 10u, Capacitor_SMD:C_0402_1005Metric
- removed C37: 10uF, Capacitor_SMD:C_0805_2012Metric
- removed J16: Conn_01x03_MountingPin, Connector_JST:JST_GH_SM03B-GHS-TB_1x03-1MP_P1.25mm_Horizontal
- removed L6: 3.3uH, Capacitor_SMD:C_0805_2012Metric_Pad1.18x1.45mm_HandSolder
- removed Q7: BSS138, Package_TO_SOT_SMD:SOT-23
- removed R40, R41: 10K, Resistor_SMD:R_0603_1608Metric_Pad0.98x0.95mm_HandSolder
- removed U12: SAM-M8Q, RF_GPS:ublox_SAM-M8Q
- added C39: 10uF, Capacitor_SMD:C_0805_2012Metric, F.Cu at (118.8, 32.7)
- added J1: NEO-6M, Connector_PinSocket_2.54mm:PinSocket_1x05_P2.54mm_Vertical, F.Cu at (194.1, 54.6)
- added J2: Conn_01x03, Connector_JST:JST_XH_B3B-XH-AM_1x03_P2.50mm_Vertical, F.Cu at (172.0, 84.0)
- added L1: 3.3uH, Inductor_SMD:L_0805_2012Metric_Pad1.05x1.20mm_HandSolder, F.Cu at (183.7, 70.1)
- added Q8: BSS138, Package_TO_SOT_SMD:SOT-23, F.Cu at (188.0, 65.2)
- added R42: 10K, Resistor_SMD:R_0603_1608Metric_Pad0.98x0.95mm_HandSolder, F.Cu at (188.0, 62.4)
- added R43: 10K, Resistor_SMD:R_0603_1608Metric_Pad0.98x0.95mm_HandSolder, F.Cu at (191.0, 65.5)
- C26, C27, C30, C31, C32, C56, C57, C58, C59, C60, C61, C62: footprint Capacitor_SMD:C_0402_1005Metric -> Capacitor_SMD:C_0201_0603Metric
- C34: value 10u -> 470uF; footprint Capacitor_SMD:C_0402_1005Metric -> Capacitor_SMD:CP_Elec_6.3x5.4_Nichicon
- moved BNO08x1 214.5 mm to (256.9, 58.1)
- moved J3 188.1 mm to (100.2, 27.4), turned to -90 degrees
- moved J9 184.6 mm to (193.4, 89.0), turned to -90 degrees
- moved J23 181.0 mm to (100.2, 34.3), turned to -90 degrees
- moved J18 170.9 mm to (194.1, 146.0), turned to 90 degrees
- moved JP6 163.1 mm to (244.7, 96.7), turned to 0 degrees
- moved U10 161.4 mm to (184.4, 145.7), turned to 90 degrees
- moved R34 158.8 mm to (104.6, 34.0), turned to 90 degrees
- moved D7 156.6 mm to (109.0, 34.5)
- moved J21 152.3 mm to (109.2, 146.9)
- moved R37 151.5 mm to (119.3, 28.1)
- moved U9 151.4 mm to (172.9, 145.7), turned to 90 degrees
- moved U23 151.4 mm to (120.4, 37.8), turned to 90 degrees
- moved R39 148.5 mm to (132.2, 25.3), turned to 0 degrees
- moved R38 147.7 mm to (133.9, 26.3), turned to -90 degrees
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Connections:
- C34 pad 1: +3V3 -> Net-(D7-A1)
- D3 pad 1: Net-(J15-Pin_1) -> Net-(J15-Pin_2)
- D3 pad 2: Net-(J15-Pin_2) -> Net-(J15-Pin_1)
- F1 pad 1: Net-(J3-Pin_2) -> Net-(J23-Pin_2)
- F1 pad 2: Net-(J23-Pin_2) -> Net-(Q2-D)
- J20 pad 1: +3V3 -> GND
- J20 pad 10: GND -> +3V3
- J26 pad 1: Net-(J26-Pin_1) -> GND
- J26 pad 2: Net-(J26-Pin_2) -> +3V3
- J26 pad 7: +3V3 -> Net-(J26-Pin_7)
- J26 pad 8: GND -> Net-(J26-Pin_8)
- J3 pad 2: Net-(J3-Pin_2) -> Net-(J23-Pin_2)
- J4 pad 2: Net-(J13-Pin_1) -> Net-(J12-Pin_1)
- J4 pad 4: Net-(J12-Pin_1) -> Net-(J13-Pin_1)
- Q2 pad 3: Net-(J23-Pin_2) -> Net-(Q2-D)
- R5 pad 1: Net-(J15-Pin_2) -> Net-(J15-Pin_1)
- R6 pad 1: Net-(J15-Pin_1) -> Net-(J15-Pin_2)
- U14 pad 10: RPI_READY -> Net-(U14-GPIO7)
- U14 pad 34: Net-(U14-GPIO22) -> RPI_READY
- U14 pad 36: Net-(J26-Pin_1) -> Net-(J26-Pin_8)
- U14 pad 37: Net-(J26-Pin_2) -> Net-(J26-Pin_7)
- U14 pad 40: Net-(J26-Pin_3) -> Net-(J26-Pin_6)
- U14 pad 41: Net-(J26-Pin_4) -> Net-(J26-Pin_5)
- U14 pad 42: Net-(J26-Pin_5) -> Net-(J26-Pin_4)
- U14 pad 43: Net-(J26-Pin_6) -> Net-(J26-Pin_3)
- U15 pad 1: ENC3A -> ENC4B
- U15 pad 10: B1_3 -> B1_4
- U15 pad 11: B1_4 -> B1_3
- U15 pad 12: B1_5 -> B1_2
- U15 pad 13: B1_6 -> B1_1
- U15 pad 14: B1_7 -> B1_0
- U15 pad 2: ENC4B -> ENC4A
- U15 pad 21: ENC2B -> ENC1A
- U15 pad 22: ENC2A -> ENC1B
- U15 pad 23: ENC1B -> ENC2A
- U15 pad 24: ENC1A -> ENC2B
- U15 pad 28: B0_3 -> B0_0
- U15 pad 29: B0_2 -> B0_1
- U15 pad 3: ENC4A -> ENC3B
- U15 pad 30: B0_7 -> B0_2
- U15 pad 31: B0_6 -> B0_3
- U15 pad 32: B0_5 -> B0_4
- U15 pad 33: B0_4 -> B0_5
- U15 pad 34: B0_0 -> B0_6
- U15 pad 35: B0_1 -> B0_7
- U15 pad 4: ENC3B -> ENC3A
- U15 pad 5: B1_0 -> B1_7
- U15 pad 8: B1_1 -> B1_6
- U15 pad 9: B1_2 -> B1_5
- U2 pad 6: Net-(J15-Pin_2) -> Net-(J15-Pin_1)
- U2 pad 7: Net-(J15-Pin_1) -> Net-(J15-Pin_2)
- U29 pad 1: Net-(U14-GPIO22) -> Net-(U14-GPIO7)
Routing:
- net +5V: track 0.00 -> 64.7 mm, vias 0 -> 2
- net MASTER_INT: track 0.00 -> 47.7 mm, vias 0 -> 2
- net SCL: track 0.00 -> 47.1 mm, vias 0 -> 2
- net VUSB: track 6.79 -> 45.9 mm, vias 0 -> 2
- net SDA: track 0.00 -> 38.6 mm, vias 0 -> 2
- net Net-(Q10-D): track 0.00 -> 34.6 mm, vias 0 -> 2
- net TX_INT: track 0.00 -> 26.9 mm, vias 0 -> 1
- net PPS: track 4.52 -> 29.5 mm, vias 0 -> 1
- net RX_INT: track 0.00 -> 23.9 mm, vias 0 -> 1
- net Net-(J12-Pin_1): track 37.0 -> 17.6 mm
- net Net-(J21-Pin_1): track 0.00 -> 19.3 mm, vias 0 -> 2
- net Net-(D7-A1): track 0.00 -> 18.8 mm
- net +1V1: track 0.00 -> 18.7 mm
- net Net-(U14-QSPI_SD3): track 0.00 -> 18.6 mm
- net Net-(J21-Pin_5): track 0.00 -> 18.4 mm, vias 0 -> 2
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- added copper zone on F.Cu, net +1V1
- added copper zone on F.Cu, net +3V3
- added copper zone on B.Cu, net GND
Other:
- copper layers 2 -> 4
- board text removed: "Encoders"
- board text removed: "Pico"

Commit message: minor changes on PCB (if any)
Parts:
- moved JP4 137.1 mm to (115.6, 135.8)
- moved BNO08x1 110.8 mm to (153.8, 98.6)
- moved R16 88.0 mm to (163.8, 108.5), turned to 180 degrees
- moved JP6 82.0 mm to (162.7, 98.5), turned to 90 degrees
- moved R21 78.9 mm to (167.2, 99.6), turned to 180 degrees
- moved SW3 78.3 mm to (164.8, 102.4), turned to 180 degrees
- moved R20 75.4 mm to (164.8, 105.4), turned to 180 degrees
- moved C12 74.8 mm to (168.2, 102.6), turned to -90 degrees
- moved C14 73.2 mm to (165.3, 107.1), turned to 180 degrees
- moved U16 72.0 mm to (171.2, 102.6), turned to 0 degrees
- moved R26 71.6 mm to (163.8, 110.6), turned to 180 degrees
- moved JP3 69.4 mm to (163.7, 113.4), turned to -90 degrees
- moved U11 69.0 mm to (168.2, 108.4), turned to -90 degrees
- moved R12 67.4 mm to (177.5, 102.1), turned to 180 degrees
- moved R19 66.4 mm to (175.1, 104.6), turned to 90 degrees
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Routing:
- net GND: track 294.2 -> 326.1 mm, vias 25 -> 29
- net SDA_OUT: track 8.43 -> 28.4 mm
- net SCL_OUT: track 3.87 -> 20.2 mm
- net Net-(JP1-B): track 17.3 -> 3.92 mm, vias 2 -> 0
- net Net-(J15-Pin_1): track 15.4 -> 27.1 mm
- net ACTIVE: track 23.4 -> 33.1 mm
- net Net-(J22-Pin_2): track 9.97 -> 19.1 mm
- net Net-(U3-OSC1): track 5.12 -> 12.4 mm, vias 0 -> 2
- net SCL: track 47.1 -> 52.8 mm, vias 2 -> 3
- net Net-(U2-RXD): track 1.86 -> 7.46 mm
- net SDA: track 38.6 -> 33.1 mm
- net Net-(J23-Pin_2): track 17.6 -> 22.9 mm
- net +5V: track 64.7 -> 69.8 mm
- net RUN: track 8.18 -> 12.1 mm
- net Net-(U4-LED0): track 21.0 -> 17.4 mm, vias 2 -> 1
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Other:
- board text removed: "PSU"
