File: titanRIO.kicad_pcb (KiCad board)
At the start: 4 copper layers, 138 parts, among them J1 NEO-6M, J10 Conn_01x04, J12 Conn_01x10, J13 Conn_01x10, J15 Screw_Terminal_01x02, J17 USB_C_Receptacle_USB2.0_16P, J18 Screw_Terminal_01x02, J2 Conn_01x03, J20 Conn_01x10, J21 Conn_01x08, J22 Conn_01x02, J23 Screw_Terminal_01x02, J24 Conn_01x12, J26 Conn_01x08, J3 Screw_Terminal_01x02, J4 Conn_02x02_Odd_Even, J5 Screw_Terminal_01x02, J6 Conn_01x04, J7 Screw_Terminal_01x02, J9 Conn_01x05, Q10 BSS138, Q11 BSS138, Q2 DMP3099L, Q4 BSS138, Q8 BSS138, SW2 SW_DIP_x03, SW3 SW_Push, SW6 SW_Push, U11 74LVC2G08, U14 RP2350A-QFN60, U15 Tang_Nano_20K, U16 74LVC1G175, U17 74HC123, U19 DAC6578xPW, U2 TCAN332G, U21 W25Q128JVS, U23 INA219AxD, U25 AP63203WU, U26 AP63205WU, U27 TPS2116DRL, U29 MB85RS256B, U3 MCP2518FD-xQBB, U4 PCA9685BS, U5 SN74LVC8T245PWR, U6 SN74LVC8T245PWR, Y1 20mHz, Y2 SG-3031CM, Y5 12MHz

Commit message: PSU redesign, or so I tried
Parts:
- C34: footprint Capacitor_SMD:CP_Elec_6.3x5.4_Nichicon -> Capacitor_SMD:CP_Elec_8x10
- moved C43 20.7 mm to (124.0, 61.4), turned to 0 degrees
- moved D15 20.5 mm to (144.4, 53.3), turned to -90 degrees
- moved D16 19.3 mm to (150.4, 53.3), turned to -90 degrees
- moved Q2 19.1 mm to (108.2, 53.3), turned to 180 degrees
- moved D9 19.0 mm to (147.4, 53.3), turned to -90 degrees
- moved BZ2 18.9 mm to (138.3, 71.1)
- moved R38 18.0 mm to (128.0, 59.6)
- moved U27 17.4 mm to (129.9, 59.6), turned to -90 degrees
- moved U25 16.9 mm to (129.8, 55.1), turned to 0 degrees
- moved C44 16.5 mm to (127.1, 61.4), turned to 0 degrees
- moved U26 15.9 mm to (124.3, 64.2), turned to 0 degrees
- moved R37 15.6 mm to (117.5, 63.8)
- moved R39 15.5 mm to (128.5, 57.6), turned to 180 degrees
- moved C39 14.7 mm to (114.9, 60.1), turned to 180 degrees
- moved C41 14.6 mm to (129.2, 52.4), turned to 0 degrees
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Routing:
- net VUSB: track 46.6 -> 63.3 mm
- net GND: track 326.1 -> 314.1 mm, vias 29 -> 32
- net SCL: track 52.8 -> 43.5 mm, vias 3 -> 2
- net Net-(D7-A1): track 18.8 -> 27.8 mm
- net Net-(J23-Pin_2): track 22.9 -> 16.4 mm
- net +5V: track 69.8 -> 64.7 mm
- net +3V3: track 191.5 -> 196.6 mm
- net SDA_OUT: track 28.4 -> 23.9 mm
- net Net-(R28-Pad1): track 1.45 -> 5.55 mm
- net Net-(U26-SW): track 8.44 -> 4.41 mm
- net Net-(U25-SW): track 7.73 -> 3.99 mm
- net Net-(U23-IN-): track 5.38 -> 8.96 mm
- net Net-(Q2-D): track 7.54 -> 4.29 mm
- net /5V_REG: track 9.98 -> 12.4 mm
- net Net-(D7-A2): track 10.4 -> 8.14 mm
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
Commit message: Added edge cut and reworked safety (but not routed yet)
Parts:
- moved JP6 32.7 mm to (193.3, 118.8), turned to 0 degrees
- moved JP3 30.4 mm to (194.1, 96.4)
- moved BNO08x1 27.7 mm to (168.3, 121.4), turned to 180 degrees
- moved R26 25.4 mm to (189.9, 96.3), turned to -90 degrees
- moved R12 25.3 mm to (179.9, 127.1), turned to 90 degrees
- moved R21 24.6 mm to (176.8, 123.6), turned to -90 degrees
- moved SW3 24.2 mm to (181.8, 123.3)
- moved R19 23.6 mm to (185.8, 127.4), turned to -90 degrees
- moved Q4 22.8 mm to (182.9, 127.4), turned to 180 degrees
- moved C12 21.2 mm to (178.3, 123.1)
- moved C11 21.2 mm to (181.3, 99.9)
- moved R20 19.4 mm to (185.7, 116.5), turned to 90 degrees
- moved U16 19.2 mm to (188.6, 117.3), turned to 90 degrees
- moved R18 16.9 mm to (178.0, 100.9), turned to -90 degrees
- moved R16 16.6 mm to (182.0, 118.5)
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Routing:
- net +3V3: track 196.6 -> 76.5 mm
- net (no net): track 50.3 -> 0.00 mm
- net GND: track 314.1 -> 266.9 mm, vias 32 -> 31
- net Net-(U17A-Q): track 33.4 -> 0.00 mm
- net Net-(J7-Pin_2): track 29.2 -> 0.00 mm
- net Net-(U16-~{CLR}): track 28.2 -> 0.00 mm
- net Net-(J5-Pin_1): track 24.7 -> 0.00 mm
- net Net-(J5-Pin_2): track 26.0 -> 4.28 mm
- net ACTIVE: track 31.9 -> 22.1 mm, vias 1 -> 0
- net CLR_FAULT: track 8.22 -> 0.00 mm
- net ~{ACTIVE}: track 5.16 -> 0.00 mm, vias 1 -> 0
- net Net-(U17A-RCext): track 5.03 -> 0.00 mm
- net Net-(U17B-RCext): track 4.74 -> 0.00 mm
- net RPI_READY: track 4.68 -> 1.23 mm, vias 2 -> 1
- net WDI_MASTER: track 2.44 -> 0.00 mm, vias 1 -> 0
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Other:
- board outline added: 100 x 100 mm
- board text removed: "Safety"

Commit message: i forgor to remove the 2 in-between layers. we good now tho
Other:
- copper layers 4 -> 2

Commit message: fih
Parts:
- added G***: LOGO, LOGO, F.Cu at (178.2, 135.6)
- added G***: LOGO, LOGO, F.Cu at (157.2, 81.4)
- added kibuzzard-6AD48C4E: G***, kibuzzard-6AD48C4E, F.Cu at (148.8, 106.8)
- added kibuzzard-6AD48C85: G***, kibuzzard-6AD48C85, F.Cu at (159.9, 107.0)
- added kibuzzard-6AD48C9F: G***, kibuzzard-6AD48C9F, F.Cu at (153.7, 133.4)
Routing:
- net ACTIVE: track 22.1 -> 247.8 mm, vias 0 -> 12
- net SCL_OUT: track 20.0 -> 189.3 mm, vias 1 -> 14
- net SDA_OUT: track 23.9 -> 187.7 mm, vias 1 -> 12
- net ~{PPS}: track 3.13 -> 139.4 mm, vias 0 -> 7
- net ~{ACTIVE}: track 0.00 -> 114.8 mm, vias 0 -> 7
- net UART_RX: track 2.34 -> 114.8 mm, vias 0 -> 6
- net CAN_INT: track 2.83 -> 111.4 mm, vias 2 -> 8
- net CAN_CS: track 3.23 -> 103.0 mm, vias 1 -> 4
- net UART_TX: track 2.27 -> 100.2 mm, vias 0 -> 8
- net FPGA_SIG1: track 0.00 -> 93.6 mm, vias 0 -> 5
- net Net-(J24-Pin_10): track 0.00 -> 87.6 mm, vias 0 -> 4
- net SCK_INT: track 7.18 -> 94.6 mm, vias 1 -> 7
- net FPGA_SIG0: track 0.00 -> 80.7 mm, vias 0 -> 2
- net GND: track 266.9 -> 344.4 mm, vias 31 -> 53
- net MOSI_INT: track 8.08 -> 79.9 mm, vias 1 -> 10
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